File: PCB_filter_1tol_THT/PCB_filter_1tol_THT.kicad_pcb (KiCad board)
At the start: 2 copper layers, 26 parts, among them J1 Conn_01x02_Pin, J2 Conn_01x02_Pin, U1 AD620, U3 LF444ACN_NOPB

Commit message: last
Parts:
- removed U3: LF444ACN_NOPB, LF444ACN_NOPB:DIP245762X508-14
- added U2: LM2902N/NOPB, LM2902N:NFF_14, F.Cu at (155.6, 120.9)
- J1: value Conn_01x02_Pin -> Conn_01x03_Pin; footprint Connector_Wire:SolderWire-0.1sqmm_1x02_P3.6mm_D0.4mm_OD1mm_Relief -> Connector_Wire:SolderWire-0.1sqmm_1x03_P3.6mm_D0.4mm_OD1mm_Relief
- moved J1 4.20 mm to (156.9, 132.3)
Routing:
- net VCC: track 77.7 -> 84.2 mm
- net GND: track 103.3 -> 109.2 mm
- net OUT3: track 10.0 -> 13.2 mm
- net IN1-: track 16.2 -> 17.1 mm
- net IN2+: track 11.9 -> 12.7 mm
- net IN3-: track 54.5 -> 53.6 mm
- net IN4+: track 17.6 -> 16.9 mm
- net IN3+: track 12.1 -> 11.4 mm

Commit message: last
Parts:
- R1, R10, R11, R12, R13, R14, R15, R2, R3, R4, R5, R6, R7, R8, R9: footprint Resistor_THT:R_Axial_DIN0207_L6.3mm_D2.5mm_P7.62mm_Horizontal -> DAVID:R_hueco_grande
- moved J2 5.02 mm to (164.2, 77.8)
Routing:
- net GND: track 109.2 -> 96.8 mm
- net Net-(J2-Pin_2): track 22.4 -> 27.4 mm
- net Net-(J2-Pin_1): track 30.7 -> 35.8 mm
- net IN1+: track 15.9 -> 16.5 mm
- added copper zone on B.Cu, net GND
- added copper zone on F.Cu, net GND
Other:
- board outline added: 30.5 x 84 mm
- board text added: "CSC - CONICET PCG-Sensor-01"
