File: PCB_filter_1tol_THT/PCB_filter_1tol_THT.kicad_sch (KiCad schematic)
At the start: 26 parts, among them J1 Conn_01x02_Pin, J2 Conn_01x02_Pin, U1 AD620, U3 LF444ACN_NOPB

Commit message: last
Parts:
- removed J1: Conn_01x02_Pin, Connector_Wire:SolderWire-0.1sqmm_1x02_P3.6mm_D0.4mm_OD1mm_Relief, symbol Connector:Conn_01x02_Pin
- added J1: Conn_01x03_Pin, Connector_Wire:SolderWire-0.1sqmm_1x03_P3.6mm_D0.4mm_OD1mm_Relief, symbol Connector:Conn_01x03_Pin
- added U2: LM2902N/NOPB, NFF_14, symbol LM2902N:LM2902N_NOPB
Connections:
- net GND: now also J1.2 (Pin_2), U2.11 (GND)
- net IN1+: now also U2.3 (INPUT1+)
- net IN1-: now also U2.1 (OUTPUT1), U2.2 (INPUT1-)
- net IN2+: now also U2.5 (INPUT2+)
- net IN2-: now also U2.6 (INPUT2-), U2.7 (OUTPUT2)
- net IN3+: now also U2.10 (INPUT3+)
- net IN3-: now also U2.9 (INPUT3-)
- net IN4+: now also U2.12 (INPUT4+)
- net OUT3: now also J1.3 (Pin_3), U2.8 (OUTPUT3)
- net VCC: now also J1.1 (Pin_1), U2.4 (V+)
- net VGND: now also U2.13 (INPUT4-), U2.14 (OUTPUT4)

Commit message: last
Parts:
- removed U3: LF444ACN_NOPB, LF444ACN_NOPB:DIP245762X508-14, symbol LF444ACN_NOPB:LF444ACN_NOPB
- R1, R10, R11, R12, R13, R14, R15, R2, R3, R4, R5, R6, R7, R8, R9: footprint Resistor_THT:R_Axial_DIN0207_L6.3mm_D2.5mm_P7.62mm_Horizontal -> DAVID:R_hueco_grande
- U2: footprint NFF_14 -> LM2902N:NFF_14
